Commit message: update

File: rotors_description/urdf/component_snippets.xacro (robot description, xacro)
@@ -747,5 +747,5 @@
       parent_link="${namespace}/vi_sensor_link"
       imu_topic="imu"
-      mass_imu_sensor="0.015"
+      mass_imu_sensor="0.00001"
       gyroscope_noise_density="0.0003394"
       gyroscope_random_walk="0.000038785"
@@ -757,5 +757,5 @@
       accelerometer_turn_on_bias_sigma="0.1960">
       <inertia ixx="0.00001" ixy="0.0" ixz="0.0" iyy="0.00001" iyz="0.0" izz="0.00001" />
-      <origin xyz="0.015 0 0.0113" rpy="0 0 0" />
+      <origin xyz="0.0 0 0.0" rpy="0 0 0" />
     </xacro:imu_plugin_macro>
   </xacro:macro>
